File: hardware/control_in.kicad_sch (KiCad schematic)
At the start: 2 parts

Commit message: Via spamming #1
Parts:
- JCNTL1, JCNTL2: Characteristics (none) -> Headers & Wire Housings Shrouded Terminal Strip, 0.050"(1.2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; Package (none) -> Other
Changed lines of the file:
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@@
   (title_block
     (title "Control In / Power Out")
-    (date "2023-01-26")
-    (rev "0.0.10")
+    (date "2023-02-08")
+    (rev "0.0.11")
     (comment 2 "http://creativecommons.org/licenses/by-sa/4.0/")
     (comment 3 "License: CC By SA 4.0")
@@
   )
   (bus (pts (xy 73.66 60.96) (xy 73.66 63.5))
-    (stroke (width 0) (type default) (color 0 0 0 0))
+    (stroke (width 0) (type default) (color 255 255 0 1))
   )
   (wire (pts (xy 53.34 63.5) (xy 71.12 63.5))
@@
   )
   (bus (pts (xy 73.66 58.42) (xy 73.66 60.96))
-    (stroke (width 0) (type default) (color 0 0 0 0))
+    (stroke (width 0) (type default) (color 255 255 0 1))
   )
   (bus (pts (xy 73.66 71.12) (xy 88.9 71.12))
-    (stroke (width 0) (type default) (color 0 0 0 0))
+    (stroke (width 0) (type default) (color 255 255 0 1))
   )
   (wire (pts (xy 53.34 86.36) (xy 71.12 86.36))
@@
   )
   (bus (pts (xy 73.66 78.74) (xy 73.66 83.82))
-    (stroke (width 0) (type default) (color 0 0 0 0))
+    (stroke (width 0) (type default) (color 255 255 0 1))
   )
   (wire (pts (xy 71.12 91.44) (xy 53.34 91.44))
@@
   )
   (bus (pts (xy 73.66 83.82) (xy 73.66 86.36))
-    (stroke (width 0) (type default) (color 0 0 0 0))
+    (stroke (width 0) (type default) (color 255 255 0 1))
   )
   (wire (pts (xy 39.37 63.5) (xy 39.37 68.834))
@@
   )
   (bus (pts (xy 73.66 86.36) (xy 73.66 88.9))
-    (stroke (width 0) (type default) (color 0 0 0 0))
+    (stroke (width 0) (type default) (color 255 255 0 1))
   )
   (wire (pts (xy 39.37 96.52) (xy 39.37 104.14))
@@
   )
   (bus (pts (xy 73.66 63.5) (xy 73.66 66.04))
-    (stroke (width 0) (type default) (color 0 0 0 0))
+    (stroke (width 0) (type default) (color 255 255 0 1))
   )
   (wire (pts (xy 71.12 88.9) (xy 53.34 88.9))
@@
   )
   (bus (pts (xy 73.66 66.04) (xy 73.66 71.12))
-    (stroke (width 0) (type default) (color 0 0 0 0))
+    (stroke (width 0) (type default) (color 255 255 0 1))
   )
   (bus (pts (xy 73.66 88.9) (xy 73.66 91.44))
-    (stroke (width 0) (type default) (color 0 0 0 0))
+    (stroke (width 0) (type default) (color 255 255 0 1))
   )
   (bus (pts (xy 88.9 78.74) (xy 73.66 78.74))
-    (stroke (width 0) (type default) (color 0 0 0 0))
+    (stroke (width 0) (type default) (color 255 255 0 1))
   )
   (wire (pts (xy 39.37 60.96) (xy 39.37 63.5))
@@
     (effects (font (size 1.27 1.27) bold) (justify right bottom))
   )
-  (global_label "+BATT" (shape input) (at 76.2 96.52 0) (fields_autoplaced)
-    (effects (font (size 1.27 1.27) bold) (justify left))
-    (property "Intersheet References" "${INTERSHEET_REFS}" (id 0) (at 84.6697 96.393 0)
-      (effects (font (size 1.27 1.27) bold) (justify left) hide)
-    )
-  )
-  (global_label "+BATT" (shape input) (at 76.2 53.34 0) (fields_autoplaced)
-    (effects (font (size 1.27 1.27) bold) (justify left))
-    (property "Intersheet References" "${INTERSHEET_REFS}" (id 0) (at 84.6697 53.213 0)
-      (effects (font (size 1.27 1.27) bold) (justify left) hide)
-    )
+  (hierarchical_label "+BATT" (shape input) (at 76.2 53.34 0)
+    (effects (font (size 2 2) bold) (justify left))
   )
   (hierarchical_label "BANK_B{CNTL[5..8]}" (shape output) (at 88.9 78.74 0)
@@
   )
   (hierarchical_label "BANK_A{CNTL[1..4]}" (shape output) (at 88.9 71.12 0)
+    (effects (font (size 2 2) bold) (justify left))
+  )
+  (hierarchical_label "+BATT" (shape input) (at 76.2 96.52 0)
     (effects (font (size 2 2) bold) (justify left))
   )
@@
     (property "Mouser Price/Stock" "https://www.mouser.com/ProductDetail/Samtec/SHF-105-01-L-D-RA-TR?qs=%252BZP6%2F%252BtExtA3jdVUpsGHlg%3D%3D" (id 11) (at 46.355 128.27 0)
       (effects (font (size 1.27 1.27)) (justify left bottom) hide)
+    )
+    (property "Characteristics" "Headers & Wire Housings Shrouded Terminal Strip, 0.050\"(1.27mm) pitch, Pin(Male), Right Angle, IDC; 10 Pos. 2 Rows;" (id 12) (at 46.355 91.44 0)
+      (effects (font (size 1.27 1.27)) hide)
+    )
+    (property "Package" "Other" (id 13) (at 46.355 91.44 0)
+      (effects (font (size 1.27 1.27)) hide)
     )
     (pin "1")
@@
       (effects (font (size 1.27 1.27)) (justify left bottom) hide)
     )
+    (property "Characteristics" "Headers & Wire Housings Shrouded Terminal Strip, 0.050\"(1.27mm) pitch, Pin(Male), Right Angle, IDC; 10 Pos. 2 Rows;" (id 12) (at 46.355 58.42 0)
+      (effects (font (size 1.27 1.27)) hide)
+    )
+    (property "Package" "Other" (id 13) (at 46.355 58.42 0)
+      (effects (font (size 1.27 1.27)) hide)
+    )
     (pin "1")

Commit message: Pre KiCad 7.0.0 WIP
Parts:
- JCNTL1, JCNTL2: MFP (none) -> SHF-105-01-L-D-RA
Connections:
- net BANK_A.CNTL1 renamed BANK_A.OUT1
- net BANK_A.CNTL2 renamed BANK_A.OUT2
- net BANK_A.CNTL3 renamed BANK_A.OUT3
- net BANK_A.CNTL4 renamed BANK_A.OUT4
- net BANK_B.CNTL5 renamed BANK_B.OUT5
- net BANK_B.CNTL6 renamed BANK_B.OUT6
- net BANK_B.CNTL7 renamed BANK_B.OUT7
- net BANK_B.CNTL8 renamed BANK_B.OUT8
Changed lines of the file:
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@@
     (effects (font (size 4 4) bold italic) (justify left bottom))
   )
-  (label "BANK_B.CNTL7" (at 71.12 88.9 180)
+  (label "BANK_B.OUT7" (at 71.12 88.9 180)
     (effects (font (size 1.27 1.27)) (justify right bottom))
   )
-  (label "BANK_A.CNTL1" (at 71.12 55.88 180)
+  (label "BANK_A.OUT1" (at 71.12 55.88 180)
     (effects (font (size 1.27 1.27) bold) (justify right bottom))
   )
-  (label "BANK_B.CNTL8" (at 71.12 86.36 180)
+  (label "BANK_B.OUT8" (at 71.12 86.36 180)
     (effects (font (size 1.27 1.27)) (justify right bottom))
   )
-  (label "BANK_B.CNTL6" (at 71.12 91.44 180)
+  (label "BANK_B.OUT6" (at 71.12 91.44 180)
     (effects (font (size 1.27 1.27)) (justify right bottom))
   )
-  (label "BANK_A.CNTL4" (at 71.12 63.5 180)
+  (label "BANK_A.OUT4" (at 71.12 63.5 180)
     (effects (font (size 1.27 1.27) bold) (justify right bottom))
   )
-  (label "BANK_A.CNTL3" (at 71.12 60.96 180)
+  (label "BANK_A.OUT3" (at 71.12 60.96 180)
     (effects (font (size 1.27 1.27) bold) (justify right bottom))
   )
-  (label "BANK_B.CNTL5" (at 71.12 93.98 180)
+  (label "BANK_B.OUT5" (at 71.12 93.98 180)
     (effects (font (size 1.27 1.27)) (justify right bottom))
   )
-  (label "BANK_A.CNTL2" (at 71.12 58.42 180)
+  (label "BANK_A.OUT2" (at 71.12 58.42 180)
     (effects (font (size 1.27 1.27) bold) (justify right bottom))
   )
@@
     (effects (font (size 2 2) bold) (justify left))
   )
-  (hierarchical_label "BANK_B{CNTL[5..8]}" (shape output) (at 88.9 78.74 0)
+  (hierarchical_label "BANK_B{OUT[5..8]}" (shape output) (at 88.9 78.74 0)
     (effects (font (size 2 2) (thickness 0.4) bold) (justify left))
   )
-  (hierarchical_label "BANK_A{CNTL[1..4]}" (shape output) (at 88.9 71.12 0)
+  (hierarchical_label "BANK_A{OUT[1..4]}" (shape output) (at 88.9 71.12 0)
     (effects (font (size 2 2) bold) (justify left))
   )
@@
     )
     (property "Package" "Other" (id 13) (at 46.355 91.44 0)
+      (effects (font (size 1.27 1.27)) hide)
+    )
+    (property "MFP" "SHF-105-01-L-D-RA" (id 14) (at 46.355 91.44 0)
       (effects (font (size 1.27 1.27)) hide)
     )
@@
       (effects (font (size 1.27 1.27)) hide)
     )
+    (property "MFP" "SHF-105-01-L-D-RA" (id 14) (at 46.355 58.42 0)
+      (effects (font (size 1.27 1.27)) hide)
+    )

Commit message: Commit before removing git submodules
Parts:
- JCNTL1, JCNTL2: Characteristics Headers & Wire Housings Shrouded Terminal Strip, 0.050"(1.2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 -> (none); MFP SHF-105-01-L-D-RA -> SHF-105-01-L-D-RA-TR; Package Other -> (none)
