File: hardware/power_in.kicad_sch (KiCad schematic)
At the start: 10 parts, among them M1 Fan, M2 Fan

Commit message: Via spamming #1
Parts:
- JP2: Characteristics (none) -> Pin Header; 1mm 1x2 Vertical
- LEDP1: Color (Green) -> (none)
- M1, M2: Characteristics (none) -> Pin Header; 2.54mm 1x2 Vertical; Package (none) -> Other; Type (none) -> THT
- R1: value 680 -> 680R; footprint dragon_mobile:RESC2012X65N -> Resistor_SMD:R_0805_2012Metric; symbol dragon_mobile:SDR10EZPJ152 -> dragon_mobile:680R; Characteristics Thick Film Resistor – 680Ω 5% 500mW; Anti Surge AEC-Q200; 2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 -> Thick Film Resistors 680Ohms, 5%, 500mW, Anti-Surge, SMD 08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
- TVSP1: value SM6T16V5AY -> SM6T18AY; footprint dragon_mobile:SMBJ36CATR -> dragon_mobile:SM6T18AY; symbol dragon_mobile:SM6T33AY -> dragon_mobile:SM6T18AY; Characteristics Uni-Directional TVS Diode, 16V breakdown, 600W peak, 2-Pin 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 -> Uni-Directional TVS Diode, 15.3V Working, 17.1V breakdown, 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; MFP SM6T16V5AY -> SM6T18AY; Mouser Part Number 511-SM6T16V5AY -> 511-SM6T18AY; Mouser Price/Stock https://www.mouser.com/ProductDetail/STMicroelectronics/SM6T16V5AY?qs=Ok1pvOkw6%2FqerKXvbVNOWA%3D%3D -> https://www.mouser.com/ProductDetail/STMicroelectronics/SM6T18AY?qs=94V4QatVK%252BcDIsO0p2IEXQ%3D%3D
- TVSP2: value SM6T16V5AY -> SM6T18AY; footprint dragon_mobile:SMBJ36CATR -> dragon_mobile:SM6T18AY; symbol dragon_mobile:SM6T33AY -> dragon_mobile:SM6T18AY; Characteristics Uni-Directional TVS Diode, 16V breakdown, 600W peak, 2-Pin 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 -> Uni-Directional TVS Diode, 15.3V Working, 17.1V breakdown, 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; MFP SM6T16V5AY -> SM6T18AY; Mouser Part Number 511-SM6T16V5AY -> 511-SM6T18AY; Mouser Price/Stock https://www.mouser.com/ProductDetail/STMicroelectronics/SM6T16V5AY?qs=Ok1pvOkw6%2FqerKXvbVNOWA%3D%3D -> https://www.mouser.com/ProductDetail/STMicroelectronics/SM6T18AY?qs=94V4QatVK%252BcDIsO0p2IEXQ%3D%3D; Your Instructions/Notes Reverse (Back) side mounted -> (none)
Other:
- note added: "+12-15 Volts DC"
- note removed: "+12-14 Volts DC"

Commit message: Pre KiCad 7.0.0 WIP
Parts:
- JPWR1, JPWR2: Characteristics PCB Socket; XT60; Pins: 2 Male; Color: yellow; Horizontal T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 -> (none); Height (none) -> 8.4; Height (mm) 8.40 -> (none); MFN Changzou Amass Elec -> (none); MFP XT60PW-M -> (none); Manufacturer_Name (none) -> Changzou Amass Elec; Manufacturer_Part_Number (none) -> XT60PW-M; Package Other -> (none); Type THT -> (none)
- renumbered LEDP1 to LP1
Other:
- note added: "Note: Only one of JP2 or LP1 should be used"
- note removed: "Note: Only one of JP2 or LEDP1 should be used"
Changed lines of the file:
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@@
     (effects (font (size 4 4) bold) (justify left bottom))
   )
-  (text "Note: Only one of JP2 or LEDP1 should be used" (at 132.08 66.04 0)
+  (text "Note: Only one of JP2 or LP1 should be used" (at 132.08 66.04 0)
     (effects (font (size 1.27 1.27) italic) (justify left bottom))
   )
@@
     (pin "2")
   )
-  (symbol (lib_name "XT60PW-M_1") (lib_id "dragon_mobile:XT60PW-M") (at 43.18 73.66 0) (unit 1)
+  (symbol (lib_id "dragon_mobile:XT60PW-M") (at 43.18 73.66 0) (unit 1)
     (in_bom yes) (on_board yes)
     (property "Reference" "JPWR2" (id 0) (at 43.18 68.834 0))
@@
       (effects (font (size 1.27 1.27)) (justify left) hide)
     )
-    (property "Datasheet" "https://www.tme.com/Document/9b8d0c5eb7094295f3d3112c214d3ade/XT60PW%20SPEC.pdf" (id 3) (at 43.18 88.9 0)
-      (effects (font (size 1.27 1.27)) (justify left) hide)
-    )
-    (property "Description" "PCB Socket; XT60; Pins: 2 Male; Color: yellow; Horizontal Through Hole" (id 4) (at 43.18 91.44 0)
-      (effects (font (size 1.27 1.27)) (justify left) hide)
-    )
-    (property "MFN" "Changzou Amass Elec" (id 12) (at 43.18 93.98 0)
-      (effects (font (size 1.27 1.27)) (justify left) hide)
-    )
-    (property "MFP" "XT60PW-M" (id 13) (at 43.18 96.52 0)
-      (effects (font (size 1.27 1.27)) (justify left) hide)
-    )
-    (property "Package" "Other" (id 14) (at 43.18 99.06 0)
-      (effects (font (size 1.27 1.27)) (justify left) hide)
-    )
-    (property "Type" "THT" (id 15) (at 43.18 101.6 0)
-      (effects (font (size 1.27 1.27)) (justify left) hide)
-    )
-    (property "Your Instructions/Notes" "~" (id 18) (at 43.18 104.14 0)
-      (effects (font (size 1.27 1.27)) (justify left) hide)
-    )
-    (property "Characteristics" "PCB Socket; XT60; Pins: 2 Male; Color: yellow; Horizontal Through Hole" (id 16) (at 43.18 107.95 0)
-      (effects (font (size 1.27 1.27)) (justify left) hide)
-    )
-    (property "Height (mm)" "8.40" (id 17) (at 43.18 106.045 0)
-      (effects (font (size 1.27 1.27)) (justify left) hide)
-    )
-    (property "Mouser Part Number" "~" (id 8) (at 59.69 86.36 0)
-      (effects (font (size 1.27 1.27)) (justify left) hide)
-    )
-    (property "Mouser Price/Stock" "~" (id 9) (at 43.18 110.49 0)
+    (property "Datasheet" "https://www.tme.eu/Document/9b8d0c5eb7094295f3d3112c214d3ade/XT60PW%20SPEC.pdf" (id 3) (at 43.18 88.9 0)
+      (effects (font (size 1.27 1.27)) (justify left) hide)
+    )
+    (property "Description" "Socket; DC supply; XT60; male; PIN: 2; on PCBs; THT; Colour: yellow" (id 4) (at 43.18 91.44 0)
+      (effects (font (size 1.27 1.27)) (justify left) hide)
+    )
+    (property "Mouser Part Number" "" (id 8) (at 59.69 86.36 0)
+      (effects (font (size 1.27 1.27)) (justify left) hide)
+    )
+    (property "Mouser Price/Stock" "" (id 9) (at 43.18 110.49 0)
       (effects (font (size 1.27 1.27)) (justify left) hide)
     )
     (property "Arrow Price/Stock" "" (id 19) (at 59.69 93.98 0)
+      (effects (font (size 1.27 1.27)) (justify left) hide)
+    )
+    (property "Height" "8.4" (id 8) (at 59.69 92.71 0)
+      (effects (font (size 1.27 1.27)) (justify left) hide)
+    )
+    (property "Manufacturer_Name" "Changzou Amass Elec" (id 9) (at 59.69 95.25 0)
+      (effects (font (size 1.27 1.27)) (justify left) hide)
+    )
+    (property "Manufacturer_Part_Number" "XT60PW-M" (id 10) (at 59.69 97.79 0)
+      (effects (font (size 1.27 1.27)) (justify left) hide)
+    )
+    (property "Arrow Part Number" "" (id 11) (at 59.69 91.44 0)
       (effects (font (size 1.27 1.27)) (justify left) hide)
     )
@@
   (symbol (lib_id "dragon_mobile:LTST-C190KGKT") (at 129.54 58.42 0) (mirror y) (unit 1)
     (in_bom yes) (on_board yes)
-    (property "Reference" "LEDP1" (id 0) (at 127.254 50.038 0))
+    (property "Reference" "LP1" (id 0) (at 127.254 50.038 0))
     (property "Value" "LTST-C190KGKT" (id 1) (at 127.0254 50.8 0)
       (effects (font (size 1.27 1.27)) hide)
@@
       (effects (font (size 1.27 1.27)) (justify left) hide)
     )
-    (property "Datasheet" "https://www.tme.com/Document/9b8d0c5eb7094295f3d3112c214d3ade/XT60PW%20SPEC.pdf" (id 3) (at 59.69 67.31 0)
-      (effects (font (size 1.27 1.27)) (justify left) hide)
-    )
-    (property "Description" "PCB Socket; XT60; Pins: 2 Male; Color: yellow; Horizontal Through Hole" (id 4) (at 59.69 69.85 0)
-      (effects (font (size 1.27 1.27)) (justify left) hide)
-    )
-    (property "MFN" "Changzou Amass Elec" (id 12) (at 43.18 53.34 0)
-      (effects (font (size 1.27 1.27)) hide)
-    )
-    (property "MFP" "XT60PW-M" (id 13) (at 43.18 53.34 0)
-      (effects (font (size 1.27 1.27)) hide)
-    )
-    (property "Package" "Other" (id 14) (at 43.18 53.34 0)
-      (effects (font (size 1.27 1.27)) hide)
-    )
-    (property "Type" "THT" (id 15) (at 43.18 53.34 0)
-      (effects (font (size 1.27 1.27)) hide)
-    )
-    (property "Your Instructions/Notes" "~" (id 18) (at 43.18 53.34 0)
-      (effects (font (size 1.27 1.27)) hide)
-    )
-    (property "Characteristics" "PCB Socket; XT60; Pins: 2 Male; Color: yellow; Horizontal Through Hole" (id 16) (at 43.18 53.34 0)
-      (effects (font (size 1.27 1.27)) hide)
-    )
-    (property "Height (mm)" "8.40" (id 17) (at 43.18 53.34 0)
-      (effects (font (size 1.27 1.27)) hide)
-    )
-    (property "Mouser Part Number" "~" (id 8) (at 59.69 66.04 0)
-      (effects (font (size 1.27 1.27)) (justify left) hide)
-    )
-    (property "Mouser Price/Stock" "~" (id 9) (at 59.69 68.58 0)
-      (effects (font (size 1.27 1.27)) (justify left) hide)
-    )
+    (property "Datasheet" "https://www.tme.eu/Document/9b8d0c5eb7094295f3d3112c214d3ade/XT60PW%20SPEC.pdf" (id 3) (at 59.69 67.31 0)
+      (effects (font (size 1.27 1.27)) (justify left) hide)
+    )
+    (property "Description" "Socket; DC supply; XT60; male; PIN: 2; on PCBs; THT; Colour: yellow" (id 4) (at 59.69 69.85 0)
+      (effects (font (size 1.27 1.27)) (justify left) hide)
+    )
+    (property "Mouser Part Number" "" (id 8) (at 59.69 66.04 0)
+      (effects (font (size 1.27 1.27)) (justify left) hide)
+    )
+    (property "Mouser Price/Stock" "" (id 9) (at 59.69 68.58 0)
+      (effects (font (size 1.27 1.27)) (justify left) hide)
+    )
+    (property "Height" "8.4" (id 7) (at 59.69 72.39 0)
+      (effects (font (size 1.27 1.27)) (justify left) hide)
+    )
+    (property "Manufacturer_Name" "Changzou Amass Elec" (id 8) (at 59.69 74.93 0)
+      (effects (font (size 1.27 1.27)) (justify left) hide)
+    )
+    (property "Manufacturer_Part_Number" "XT60PW-M" (id 9) (at 59.69 77.47 0)
+      (effects (font (size 1.27 1.27)) (justify left) hide)
+    )
+    (property "Arrow Part Number" "" (id 10) (at 59.69 71.12 0)
+      (effects (font (size 1.27 1.27)) (justify left) hide)
+    )
+    (property "Arrow Price/Stock" "" (id 11) (at 59.69 73.66 0)
+      (effects (font (size 1.27 1.27)) (justify left) hide)
+    )

Commit message: Commit before removing git submodules
Parts:
- JPWR1, JPWR2: Height 8.4 -> (none); Height (mm) (none) -> 8.4; MFN (none) -> Changzou Amass Elec; MFP (none) -> XT60PW-M; Manufacturer_Name Changzou Amass Elec -> (none); Manufacturer_Part_Number XT60PW-M -> (none)
- LP1: Color (none) -> (Green)
- R1: Package 0805 -> (none); Type SMD -> (none)
