File: hardware/solid_state_relays_12v.kicad_sch (KiCad schematic)
At the start: 16 parts

Commit message: Pre KiCad 7.0.0 WIP
Other:
- sheet Control In - Power Out ports: added BANK_A{OUT[1..4]}, BANK_B{OUT[5..8]}; removed BANK_A{CNTL[1..4]}, BANK_B{CNTL[5..8]}
- sheet Solid State Relays - Bank A ports: added BANK_A{OUT[1..4]}; removed BANK_A{CNTL[1..4]}
- sheet Solid State Relays - Bank B ports: added BANK_B{OUT[5..8]}; removed BANK_B{CNTL[5..8]}
Changed lines of the file:
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@@
       (effects (font (size 1.27 1.27)) (justify left top))
     )
-    (pin "BANK_B{CNTL[5..8]}" input (at 142.24 73.66 180)
+    (pin "BANK_B{OUT[5..8]}" input (at 142.24 73.66 180)
       (effects (font (size 1.27 1.27)) (justify left))
     )
@@
       (effects (font (size 1.27 1.27)) (justify left top))
     )
-    (pin "BANK_A{CNTL[1..4]}" input (at 142.24 53.34 180)
+    (pin "BANK_A{OUT[1..4]}" input (at 142.24 53.34 180)
       (effects (font (size 1.27 1.27)) (justify left))
     )
@@
       (effects (font (size 1.27 1.27)) (justify left top))
     )
-    (pin "BANK_B{CNTL[5..8]}" output (at 121.92 73.66 0)
+    (pin "BANK_B{OUT[5..8]}" output (at 121.92 73.66 0)
       (effects (font (size 1.27 1.27)) (justify right))
     )
-    (pin "BANK_A{CNTL[1..4]}" output (at 121.92 53.34 0)
+    (pin "BANK_A{OUT[1..4]}" output (at 121.92 53.34 0)
       (effects (font (size 1.27 1.27)) (justify right))
     )
@@
       (reference "JPWR2") (unit 1) (value "XT60PW-M") (footprint "dragon_mobile:XT60PWM")
     )
+    (path "/4223877a-f0b6-4f15-8613-23d3b27ad879/98df94df-9072-4d30-8bf8-f0de70bd3c38"
+      (reference "LP1") (unit 1) (value "LTST-C190KGKT") (footprint "dragon_mobile:LEDC1608X80N")
+    )
     (path "/f8ae6d4d-7a26-4f24-b773-fe0ae5d07268/a42411c5-99ce-4df7-a163-79a2fe583b5d"
-      (reference "LED1") (unit 1) (value "LTST-C190KFKT") (footprint "dragon_mobile:LEDC1607X80N")
+      (reference "LT1") (unit 1) (value "LTST-C190KFKT") (footprint "dragon_mobile:LEDC1607X80N")
     )
     (path "/f8ae6d4d-7a26-4f24-b773-fe0ae5d07268/af1a8689-fd14-4e6d-8121-0bcb7b1e9b4b"
-      (reference "LED2") (unit 1) (value "LTST-C190KFKT") (footprint "dragon_mobile:LEDC1607X80N")
+      (reference "LT2") (unit 1) (value "LTST-C190KFKT") (footprint "dragon_mobile:LEDC1607X80N")
     )
     (path "/f8ae6d4d-7a26-4f24-b773-fe0ae5d07268/07c70024-2563-419d-9d20-8731970eb9c7"
-      (reference "LED3") (unit 1) (value "LTST-C190KFKT") (footprint "dragon_mobile:LEDC1607X80N")
+      (reference "LT3") (unit 1) (value "LTST-C190KFKT") (footprint "dragon_mobile:LEDC1607X80N")
     )
     (path "/f8ae6d4d-7a26-4f24-b773-fe0ae5d07268/e6189137-bded-45c9-8a2d-c03c9bb00a13"
-      (reference "LED4") (unit 1) (value "LTST-C190KFKT") (footprint "dragon_mobile:LEDC1607X80N")
+      (reference "LT4") (unit 1) (value "LTST-C190KFKT") (footprint "dragon_mobile:LEDC1607X80N")
     )
     (path "/9aae0e2a-06c5-4008-ba6f-da2f507b83a6/8bcbf4ff-74bf-48f3-9858-b163c117f21e"
-      (reference "LED5") (unit 1) (value "LTST-C190KFKT") (footprint "dragon_mobile:LEDC1607X80N")
+      (reference "LT5") (unit 1) (value "LTST-C190KFKT") (footprint "dragon_mobile:LEDC1607X80N")
     )
     (path "/9aae0e2a-06c5-4008-ba6f-da2f507b83a6/57132f61-2128-4144-9b03-bd0d018e3901"
-      (reference "LED6") (unit 1) (value "LTST-C190KFKT") (footprint "dragon_mobile:LEDC1607X80N")
+      (reference "LT6") (unit 1) (value "LTST-C190KFKT") (footprint "dragon_mobile:LEDC1607X80N")
     )
     (path "/9aae0e2a-06c5-4008-ba6f-da2f507b83a6/694a1507-4e9e-41d3-b13b-11b431b27bf2"
-      (reference "LED7") (unit 1) (value "LTST-C190KFKT") (footprint "dragon_mobile:LEDC1607X80N")
+      (reference "LT7") (unit 1) (value "LTST-C190KFKT") (footprint "dragon_mobile:LEDC1607X80N")
     )
     (path "/9aae0e2a-06c5-4008-ba6f-da2f507b83a6/d46e7bc8-9768-4016-81b1-b9a09b537892"
-      (reference "LED8") (unit 1) (value "LTST-C190KFKT") (footprint "dragon_mobile:LEDC1607X80N")
-    )
-    (path "/4223877a-f0b6-4f15-8613-23d3b27ad879/98df94df-9072-4d30-8bf8-f0de70bd3c38"
-      (reference "LEDP1") (unit 1) (value "LTST-C190KGKT") (footprint "dragon_mobile:LEDC1608X80N")
+      (reference "LT8") (unit 1) (value "LTST-C190KFKT") (footprint "dragon_mobile:LEDC1607X80N")
     )
     (path "/4223877a-f0b6-4f15-8613-23d3b27ad879/4843324d-65d7-40e8-acb1-eb41210186e8"
