File: hardware/ssr_bank_a.kicad_sch (KiCad schematic)
At the start: 28 parts, among them J1 1190297, J2 1190297, J3 1190297, J4 1190297, Q1 IRF4905PBF, Q2 IRF4905PBF, Q3 IRF4905PBF, Q4 IRF4905PBF

Commit message: Via spamming #1
Parts:
- J1, J2, J3, J4: Characteristics 2 Position Wire to Board Terminal Block Horizontal with Lev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 -> 2 Position Wire to Board Terminal Block Horizontal with Boa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
- JL1, JL2, JL3, JL4: Characteristics (none) -> Pin Header; 1mm 1x2 Vertical
- Q1, Q2, Q3, Q4: footprint dragon_mobile:TO254P469X1042X1967-3P -> dragon_mobile:IRF4905PBF; Characteristics P-channel MOSFET; IRF4905; Max: 64A 55V; TO-220AB Through H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 -> P-channel MOSFET,IRF4905 64A 55V; Package TO-220AB -> TO-220-3; Your Instructions/Notes Reverse (Back) side mounted -> (none)
- RL1, RL2, RL3, RL4: value 680 -> 680R; footprint dragon_mobile:RESC2012X65N -> Resistor_SMD:R_0805_2012Metric; symbol dragon_mobile:SDR10EZPJ152 -> dragon_mobile:680R; Characteristics Thick Film Resistor – 680Ω 5% 500mW; Anti Surge AEC-Q200; 2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 -> Thick Film Resistors 680Ohms, 5%, 500mW, Anti-Surge, SMD 08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
- RP1, RP2, RP3, RP4: footprint dragon_mobile:RESC2012X65N -> Resistor_SMD:R_0603_1608Metric
- TVS1, TVS2, TVS3, TVS4: value SM6T16V5AY -> SM6T18AY; footprint dragon_mobile:SMBJ36CATR -> dragon_mobile:SM6T18AY; symbol dragon_mobile:SM6T30AY -> dragon_mobile:SM6T18AY; Characteristics Uni-Directional TVS Diode, 16V breakdown, 600W peak, 2-Pin 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 -> Uni-Directional TVS Diode, 15.3V Working, 17.1V breakdown, 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; MFP SM6T16V5AY -> SM6T18AY; Mouser Part Number 511-SM6T16V5AY -> 511-SM6T18AY; Mouser Price/Stock https://www.mouser.com/ProductDetail/STMicroelectronics/SM6T16V5AY?qs=Ok1pvOkw6%2FqerKXvbVNOWA%3D%3D -> https://www.mouser.com/ProductDetail/STMicroelectronics/SM6T18AY?qs=94V4QatVK%252BcDIsO0p2IEXQ%3D%3D

Commit message: Pre KiCad 7.0.0 WIP
Parts:
- renumbered LED1 to LT1, LED2 to LT2, LED3 to LT3, LED4 to LT4
Connections:
- net BANK_A.CNTL1 renamed BANK_A.OUT1
- net BANK_A.CNTL2 renamed BANK_A.OUT2
- net BANK_A.CNTL3 renamed BANK_A.OUT3
- net BANK_A.CNTL4 renamed BANK_A.OUT4
Changed lines of the file:
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@@
     (effects (font (size 1.27 1.27) italic) (justify left bottom))
   )
-  (label "BANK_A.CNTL3" (at 55.88 111.76 0)
+  (label "BANK_A.OUT3" (at 55.88 111.76 0)
     (effects (font (size 1.27 1.27)) (justify left bottom))
   )
-  (label "BANK_A.CNTL2" (at 55.88 78.74 0)
+  (label "BANK_A.OUT2" (at 55.88 78.74 0)
     (effects (font (size 1.27 1.27)) (justify left bottom))
   )
-  (label "BANK_A.CNTL1" (at 55.88 45.72 0)
+  (label "BANK_A.OUT1" (at 55.88 45.72 0)
     (effects (font (size 1.27 1.27)) (justify left bottom))
   )
-  (label "BANK_A.CNTL4" (at 55.88 144.78 0)
+  (label "BANK_A.OUT4" (at 55.88 144.78 0)
     (effects (font (size 1.27 1.27)) (justify left bottom))
   )
@@
     (effects (font (size 2 2) (thickness 0.4) bold) (justify left))
   )
-  (hierarchical_label "BANK_A{CNTL[1..4]}" (shape input) (at 45.72 30.48 180)
+  (hierarchical_label "BANK_A{OUT[1..4]}" (shape input) (at 45.72 30.48 180)
     (effects (font (size 2 2)) (justify right))
   )
@@
   (symbol (lib_id "dragon_mobile:LTST-C190KFKT") (at 76.2 124.46 0) (unit 1)
     (in_bom yes) (on_board yes)
-    (property "Reference" "LED3" (id 0) (at 80.01 127 0))
+    (property "Reference" "LT3" (id 0) (at 80.01 127 0))
     (property "Value" "LTST-C190KFKT" (id 1) (at 76.2 119.38 0)
       (effects (font (size 1.27 1.27)) (justify left bottom) hide)
@@
   (symbol (lib_id "dragon_mobile:LTST-C190KFKT") (at 76.2 58.42 0) (unit 1)
     (in_bom yes) (on_board yes)
-    (property "Reference" "LED1" (id 0) (at 80.01 60.96 0))
+    (property "Reference" "LT1" (id 0) (at 80.01 60.96 0))
     (property "Value" "LTST-C190KFKT" (id 1) (at 76.2 53.34 0)
       (effects (font (size 1.27 1.27)) (justify left bottom) hide)
@@
   (symbol (lib_id "dragon_mobile:LTST-C190KFKT") (at 76.2 91.44 0) (unit 1)
     (in_bom yes) (on_board yes)
-    (property "Reference" "LED2" (id 0) (at 80.01 93.98 0))
+    (property "Reference" "LT2" (id 0) (at 80.01 93.98 0))
     (property "Value" "LTST-C190KFKT" (id 1) (at 76.2 86.36 0)
       (effects (font (size 1.27 1.27)) (justify left bottom) hide)
@@
   (symbol (lib_id "dragon_mobile:LTST-C190KFKT") (at 76.2 157.48 0) (unit 1)
     (in_bom yes) (on_board yes)
-    (property "Reference" "LED4" (id 0) (at 80.01 160.02 0))
+    (property "Reference" "LT4" (id 0) (at 80.01 160.02 0))
     (property "Value" "LTST-C190KFKT" (id 1) (at 76.2 152.4 0)
       (effects (font (size 1.27 1.27)) (justify left bottom) hide)

Commit message: Commit before removing git submodules
Parts:
- LT1, LT2, LT3, LT4: Color (none) -> (Orange)
- Q1, Q2, Q3, Q4: Characteristics P-channel MOSFET,IRF4905 64A 55V -> (none); Package TO-220-3 -> (none); Type THT -> (none)
- RL1, RL2, RL3, RL4: Package 0805 -> (none); Type SMD -> (none)
- RP1, RP2, RP3, RP4: Characteristics Thick Film Resistor - 10KΩ 5% 300mW; Anti Surge AEC-Q200; 1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 -> (none); Height (mm) 0.55 -> (none); MFN ROHM Semiconductor -> (none); MFP SDR03EZPJ103 -> (none); Mouser Part Number 755-SDR03EZPJ103 -> (none); Mouser Price/Stock https://www.mouser.com/ProductDetail/ROHM-Semiconductor/SDR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 -> (none); Package 0603 -> (none); Type SMD -> (none)
