File: hardware/ssr_bank_b.kicad_sch (KiCad schematic)
At the start: 28 parts, among them J5 1190297, J6 1190297, J7 1190297, J8 1190297, Q5 IRF4905PBF, Q6 IRF4905PBF, Q7 IRF4905PBF, Q8 IRF4905PBF

Commit message: Via spamming #1
Parts:
- J5, J6, J7, J8: Characteristics 2 Position Wire to Board Terminal Block Horizontal with Lev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 -> 2 Position Wire to Board Terminal Block Horizontal with Boa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
- JL5, JL6, JL7, JL8: Characteristics (none) -> Pin Header; 1mm 1x2 Vertical
- Q5, Q6, Q7, Q8: footprint dragon_mobile:TO254P469X1042X1967-3P -> dragon_mobile:IRF4905PBF; Characteristics P-channel MOSFET; IRF4905; Max: 64A 55V; TO-220AB Through H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 -> P-channel MOSFET,IRF4905 64A 55V; Package TO-220AB -> TO-220-3; Your Instructions/Notes Reverse (Back) side mounted -> (none)
- RL5, RL6, RL7, RL8: value 680 -> 680R; footprint dragon_mobile:RESC2012X65N -> Resistor_SMD:R_0805_2012Metric; symbol dragon_mobile:SDR10EZPJ152 -> dragon_mobile:680R; Characteristics Thick Film Resistor – 680Ω 5% 500mW; Anti Surge AEC-Q200; 2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 -> Thick Film Resistors 680Ohms, 5%, 500mW, Anti-Surge, SMD 08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
- RP5, RP6, RP7, RP8: footprint dragon_mobile:RESC2012X65N -> Resistor_SMD:R_0603_1608Metric
- TVS5, TVS6, TVS7, TVS8: value SM6T16V5AY -> SM6T18AY; footprint dragon_mobile:SMBJ36CATR -> dragon_mobile:SM6T18AY; symbol dragon_mobile:SM6T30AY -> dragon_mobile:SM6T18AY; Characteristics Uni-Directional TVS Diode, 16V breakdown, 600W peak, 2-Pin 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 -> Uni-Directional TVS Diode, 15.3V Working, 17.1V breakdown, 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; MFP SM6T16V5AY -> SM6T18AY; Mouser Part Number 511-SM6T16V5AY -> 511-SM6T18AY; Mouser Price/Stock https://www.mouser.com/ProductDetail/STMicroelectronics/SM6T16V5AY?qs=Ok1pvOkw6%2FqerKXvbVNOWA%3D%3D -> https://www.mouser.com/ProductDetail/STMicroelectronics/SM6T18AY?qs=94V4QatVK%252BcDIsO0p2IEXQ%3D%3D

Commit message: Pre KiCad 7.0.0 WIP
Parts:
- renumbered LED5 to LT5, LED6 to LT6, LED7 to LT7, LED8 to LT8
Connections:
- net BANK_B.CNTL5 renamed BANK_B.OUT5
- net BANK_B.CNTL6 renamed BANK_B.OUT6
- net BANK_B.CNTL7 renamed BANK_B.OUT7
- net BANK_B.CNTL8 renamed BANK_B.OUT8
Changed lines of the file:
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@@
     (effects (font (size 1.27 1.27) italic) (justify left bottom))
   )
-  (label "BANK_B.CNTL5" (at 55.88 45.72 0)
+  (label "BANK_B.OUT5" (at 55.88 45.72 0)
     (effects (font (size 1.27 1.27)) (justify left bottom))
   )
-  (label "BANK_B.CNTL7" (at 55.88 111.76 0)
+  (label "BANK_B.OUT7" (at 55.88 111.76 0)
     (effects (font (size 1.27 1.27)) (justify left bottom))
   )
-  (label "BANK_B.CNTL6" (at 55.88 78.74 0)
+  (label "BANK_B.OUT6" (at 55.88 78.74 0)
     (effects (font (size 1.27 1.27)) (justify left bottom))
   )
-  (label "BANK_B.CNTL8" (at 55.88 144.78 0)
+  (label "BANK_B.OUT8" (at 55.88 144.78 0)
     (effects (font (size 1.27 1.27)) (justify left bottom))
   )
@@
   (symbol (lib_id "dragon_mobile:LTST-C190KFKT") (at 76.2 91.44 0) (unit 1)
     (in_bom yes) (on_board yes)
-    (property "Reference" "LED6" (id 0) (at 80.01 93.98 0))
+    (property "Reference" "LT6" (id 0) (at 80.01 93.98 0))
     (property "Value" "LTST-C190KFKT" (id 1) (at 76.2 86.36 0)
       (effects (font (size 1.27 1.27)) (justify left bottom) hide)
@@
   (symbol (lib_id "dragon_mobile:LTST-C190KFKT") (at 76.2 124.46 0) (unit 1)
     (in_bom yes) (on_board yes)
-    (property "Reference" "LED7" (id 0) (at 80.01 127 0))
+    (property "Reference" "LT7" (id 0) (at 80.01 127 0))
     (property "Value" "LTST-C190KFKT" (id 1) (at 76.2 119.38 0)
       (effects (font (size 1.27 1.27)) (justify left bottom) hide)
@@
   (symbol (lib_id "dragon_mobile:LTST-C190KFKT") (at 76.2 58.42 0) (unit 1)
     (in_bom yes) (on_board yes)
-    (property "Reference" "LED5" (id 0) (at 80.01 60.96 0))
+    (property "Reference" "LT5" (id 0) (at 80.01 60.96 0))
     (property "Value" "LTST-C190KFKT" (id 1) (at 76.2 53.34 0)
       (effects (font (size 1.27 1.27)) (justify left bottom) hide)
@@
   (symbol (lib_id "dragon_mobile:LTST-C190KFKT") (at 76.2 157.48 0) (unit 1)
     (in_bom yes) (on_board yes)
-    (property "Reference" "LED8" (id 0) (at 80.01 160.02 0))
+    (property "Reference" "LT8" (id 0) (at 80.01 160.02 0))
     (property "Value" "LTST-C190KFKT" (id 1) (at 76.2 152.4 0)
       (effects (font (size 1.27 1.27)) (justify left bottom) hide)

Commit message: Commit before removing git submodules
Parts:
- LT5, LT6, LT7, LT8: Color (none) -> (Orange)
- Q5, Q6, Q7, Q8: Characteristics P-channel MOSFET,IRF4905 64A 55V -> (none); Package TO-220-3 -> (none); Type THT -> (none)
- RL5, RL6, RL7, RL8: Package 0805 -> (none); Type SMD -> (none)
- RP5, RP6, RP7, RP8: Characteristics Thick Film Resistor - 10KΩ 5% 300mW; Anti Surge AEC-Q200; 1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 -> (none); Height (mm) 0.55 -> (none); MFN ROHM Semiconductor -> (none); MFP SDR03EZPJ103 -> (none); Mouser Part Number 755-SDR03EZPJ103 -> (none); Mouser Price/Stock https://www.mouser.com/ProductDetail/ROHM-Semiconductor/SDR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 -> (none); Package 0603 -> (none); Type SMD -> (none)
